Commit message: feat: add gazebo plugins for 3D Lidar and cameras

File: src/drone_description/urdf/construction_drone.xacro (robot description, xacro)
@@ -3,15 +3,16 @@
   <!-- Include base and LiDAR XACROs -->
   <xacro:include filename="$(find drone_description)/urdf/drone_base.xacro"/>
-  <xacro:include filename="$(find drone_description)/urdf/airy_lidar_right.xacro"/>
-  <xacro:include filename="$(find drone_description)/urdf/airy_lidar_left.xacro"/>
+  <xacro:include filename="$(find drone_description)/urdf/airy_lidar.xacro"/>
+  <!-- <xacro:include filename="$(find drone_description)/urdf/airy_lidar_left.xacro"/> -->
   <xacro:include filename="$(find drone_description)/urdf/fisheye_camera.xacro"/>
+  <!-- <xacro:include filename="$(find drone_description)/urdf/fisheye_camera_rear.xacro"/> -->
   <!-- Instantiate base (already includes world_link and base_link) -->
   <!-- No additional instantiation needed for drone_base.xacro -->
   <!-- Instantiate LiDARs -->
-  <xacro:robosense_airy_lidar1 name="lidar_right" parent="base_link" xyz="0.122 0.0 0.18" rpy="0 0 0"/>
-  <xacro:robosense_airy_lidar2 name="lidar_left" parent="base_link" xyz="-0.122 0.0 0.18" rpy="0 0 3.14159"/>
+  <xacro:robosense_airy_lidar name="lidar_right" parent="base_link" xyz="0.122 0.0 0.18" rpy="0 0 0"/>
+  <xacro:robosense_airy_lidar name="lidar_left" parent="base_link" xyz="-0.122 0.0 0.18" rpy="0 0 3.14159"/>
   <!-- Instatiate Fisheye Cameras -->
-  <xacro:fisheye_camera name="fisheye_camera_front" parent="base_link" xyz="0.0 0.139 0.14" rpy="0 0 3.14159"/>
-  <xacro:fisheye_camera name="fisheye_camera_rear" parent="base_link" xyz="0.0 -0.139 0.14" rpy="0 0 0"/>
-  <xacro:fisheye_camera name="fisheye_camera_below" parent="base_link" xyz="0.0 0.0 0.095" rpy="1.5708 0 0"/>
+  <xacro:fisheye_camera name="fisheye_camera_front" parent="base_link" xyz="0.0 0.139 0.14" rpy="0 0 3.14159" hfov="2.094"/> <!-- 3.14159 -->
+  <xacro:fisheye_camera name="fisheye_camera_rear" parent="base_link" xyz="0.0 -0.139 0.14" rpy="0 0 0" hfov="2.094" />
+  <xacro:fisheye_camera name="fisheye_camera_below" parent="base_link" xyz="0.0 0.0 0.095" rpy="1.5708 0 0" hfov="2.094" />
 </robot>

File: src/drone_description/urdf/fisheye_camera.xacro (robot description, xacro)
@@ -1,14 +1,14 @@
 <?xml version="1.0"?>
 <robot name="fisheye_camera" xmlns:xacro="http://www.ros.org/wiki/xacro">
-  <!-- Macro for camera -->
-  <xacro:macro name="fisheye_camera" params="name parent xyz rpy">
+  <!-- Macro for wide-angle (fisheye) camera -->
+  <xacro:macro name="fisheye_camera" params="name parent xyz rpy hfov">
     <link name="${name}_link">
       <visual>
         <origin xyz="0 0 0" rpy="0 0 0"/>
         <geometry>
-          <mesh filename="package://drone_description/meshes/fisheye_camera.dae" scale="1 1 1"/> <!-- Placeholder, adjust filepath -->
+          <mesh filename="package://drone_description/meshes/fisheye_camera.dae" scale="1 1 1"/>
         </geometry>
         <material name="black">
-          <color rgba="0 0 0 1"/> <!-- Fallback if DAE lacks textures -->
+          <color rgba="0 0 0 1"/>
         </material>
       </visual>
@@ -16,10 +16,10 @@
         <origin xyz="0 0 0" rpy="0 0 0"/>
         <geometry>
-          <mesh filename="package://drone_description/meshes/fisheye_camera.dae" scale="1 1 1"/> <!-- Same mesh -->
+          <mesh filename="package://drone_description/meshes/fisheye_camera.dae" scale="1 1 1"/>
         </geometry>
       </collision>
       <inertial>
-        <mass value="0.05"/> <!-- Placeholder: 50g, adjust from CAD -->
-        <inertia ixx="0.00001" ixy="0.0" ixz="0.0" iyy="0.00001" iyz="0.0" izz="0.00001"/> <!-- Placeholder -->
+        <mass value="0.05"/>
+        <inertia ixx="0.00001" ixy="0.0" ixz="0.0" iyy="0.00001" iyz="0.0" izz="0.00001"/>
       </inertial>
     </link>
@@ -27,59 +27,33 @@
       <parent link="${parent}"/>
       <child link="${name}_link"/>
-      <origin xyz="${xyz}" rpy="${rpy}"/> <!-- Relative to base_link -->
+      <origin xyz="${xyz}" rpy="${rpy}"/>
     </joint>
-    <!-- Gazebo reference -->
+    <!-- Gazebo plugin for regular camera (not fisheye) -->
     <gazebo reference="${name}_link">
-      <sensor type="camera" name="${name}_sensor">
-        <pose>0 0 0 0 0 0</pose>
-        <visualize>true</visualize>
-        <update_rate>30</update_rate> <!-- 30Hz for camera -->
+      <sensor type="camera" name="${name}_regular_cam">
+        <pose>0 -0.5 0 0 0 -1.5708</pose>
+        <always_on>true</always_on>
+        <update_rate>30</update_rate>
         <camera>
-          <horizontal_fov>3.14159</horizontal_fov> <!-- 180° -->
+          <horizontal_fov>${hfov}</horizontal_fov>
           <image>
-            <width>1280</width>
-            <height>720</height>
+            <width>640</width>
+            <height>480</height>
             <format>R8G8B8</format>
           </image>
           <clip>
-            <near>0.01</near> <!-- 1cm -->
-            <far>100</far> <!-- 100m -->
+            <near>0.05</near>
+            <far>100</far>
           </clip>
-          <distortion>
-            <k1>0.1</k1> <!-- Placeholder fisheye distortion -->
-            <k2>0.01</k2>
-            <k3>0.0</k3>
-            <p1>0.0</p1>
-            <p2>0.0</p2>
-            <center>0.5 0.5</center>
-          </distortion>
-          <lens>
-            <type>fisheye</type>
-            <scale_to_hfov>true</scale_to_hfov>
-            <cutoff_angle>3.14159</cutoff_angle> <!-- 180° -->
-            <env_texture_size>512</env_texture_size>
-          </lens>
-          <noise>
-            <type>gaussian</type>
-            <mean>0.0</mean>
-            <stddev>0.01</stddev>
-          </noise>
         </camera>
-        <plugin name="${name}_controller" filename="libgazebo_ros_camera.so">
-          <cameraName>camera</cameraName>
+        <plugin name="${name}_camera_controller" filename="libgazebo_ros_camera.so">
+          <cameraName>${name}</cameraName>
+          <imageTopicName>${name}/image_raw</imageTopicName>
+          <cameraInfoTopicName>${name}/camera_info</cameraInfoTopicName>
           <frameName>${name}_link</frameName>
-          <imageTopicName>/${name}/image_raw</imageTopicName>
-          <cameraInfoTopicName>/${name}/camera_info</cameraInfoTopicName>
-          <hackBaseline>0.0</hackBaseline>
-          <distortionK1>0.1</distortionK1>
-          <distortionK2>0.01</distortionK2>
-          <distortionK3>0.0</distortionK3>
-          <distortionT1>0.0</distortionT1>
-          <distortionT2>0.0</distortionT2>
+          <updateRate>30.0</updateRate>
         </plugin>
       </sensor>
     </gazebo>
   </xacro:macro>
-  <!-- Instantiate camera -->
-  <!-- <xacro:camera name="camera" parent="base_link" xyz="0.1 0.0 0.4" rpy="0 0 0"/> -->
 </robot>

Commit message: feat: add different packages, develop propellers simulations in gazebo (WIP)

File: src/drone_description/urdf/construction_drone.xacro (robot description, xacro)
@@ -20,12 +20,18 @@
   <xacro:propeller name="rear_left_prop" parent="base_link" xyz="-0.105 -0.105 0.24122" rpy="0 0 0"/>
   <xacro:propeller name="rear_right_prop" parent="base_link" xyz="0.105 -0.105 0.24122" rpy="0 0 0"/>
+  <!-- Gazebo plugin to enable ROS control -->
+  <gazebo>
+    <plugin name="gazebo_ros_control" filename="libgazebo_ros_control.so">
+      <robotNamespace>/</robotNamespace>
+    </plugin>
+  </gazebo>
   <!-- Front Right Propeller Transmission -->
   <transmission name="front_right_prop_transmission">
     <type>transmission_interface/SimpleTransmission</type>
     <joint name="front_right_prop_joint">
-      <hardwareInterface>EffortJointInterface</hardwareInterface>
+      <hardwareInterface>hardware_interface/VelocityJointInterface</hardwareInterface>
     </joint>
     <actuator name="front_right_prop_motor">
-      <hardwareInterface>EffortJointInterface</hardwareInterface>
+      <hardwareInterface>hardware_interface/VelocityJointInterface</hardwareInterface>
       <mechanicalReduction>1</mechanicalReduction>
     </actuator>
@@ -35,8 +41,8 @@
     <type>transmission_interface/SimpleTransmission</type>
     <joint name="front_left_prop_joint">
-      <hardwareInterface>EffortJointInterface</hardwareInterface>
+      <hardwareInterface>hardware_interface/VelocityJointInterface</hardwareInterface>
     </joint>
     <actuator name="front_left_prop_motor">
-      <hardwareInterface>EffortJointInterface</hardwareInterface>
+      <hardwareInterface>hardware_interface/VelocityJointInterface</hardwareInterface>
       <mechanicalReduction>1</mechanicalReduction>
     </actuator>
@@ -46,8 +52,8 @@
     <type>transmission_interface/SimpleTransmission</type>
     <joint name="rear_left_prop_joint">
-      <hardwareInterface>EffortJointInterface</hardwareInterface>
+      <hardwareInterface>hardware_interface/VelocityJointInterface</hardwareInterface>
     </joint>
     <actuator name="rear_left_prop_motor">
-      <hardwareInterface>EffortJointInterface</hardwareInterface>
+      <hardwareInterface>hardware_interface/VelocityJointInterface</hardwareInterface>
       <mechanicalReduction>1</mechanicalReduction>
     </actuator>
@@ -57,8 +63,8 @@
     <type>transmission_interface/SimpleTransmission</type>
     <joint name="rear_right_prop_joint">
-      <hardwareInterface>EffortJointInterface</hardwareInterface>
+      <hardwareInterface>hardware_interface/VelocityJointInterface</hardwareInterface>
     </joint>
     <actuator name="rear_right_prop_motor">
-      <hardwareInterface>EffortJointInterface</hardwareInterface>
+      <hardwareInterface>hardware_interface/VelocityJointInterface</hardwareInterface>
       <mechanicalReduction>1</mechanicalReduction>
     </actuator>

File: src/drone_description/urdf/drone_base.xacro (robot description, xacro)
@@ -8,5 +8,5 @@
       <origin xyz="0 0 0.1" rpy="0 0 0"/>
       <geometry>
-        <mesh filename="package://drone_description/meshes/drone_base_with_motors.dae" scale="1 1 1"/> <!-- DAE mesh, assuming mm units -->
+        <mesh filename="package://drone_description/meshes/drone_base_w_motors.stl" scale="1 1 1"/> <!-- DAE mesh, assuming mm units -->
       </geometry>
       <material name="blue">
@@ -17,10 +17,10 @@
       <origin xyz="0 0 0.1" rpy="0 0 0"/>
       <geometry>
-        <mesh filename="package://drone_description/meshes/drone_base_with_motors.dae" scale="1 1 1"/>
+        <mesh filename="package://drone_description/meshes/drone_base_w_motors.stl" scale="1 1 1"/>
         <!-- <box size="0.3 0.3 0.25"/>  -->
       </geometry>
     </collision>
     <inertial>
-      <mass value="1.0"/> <!-- Placeholder: 1kg, adjust from CAD -->
+      <mass value="0.5"/> <!-- Placeholder: 1kg, adjust from CAD -->
       <inertia ixx="0.01" ixy="0.0" ixz="0.0" iyy="0.01" iyz="0.0" izz="0.01"/> <!-- Placeholder, adjust from CAD -->
     </inertial>

Commit message: feat: add libLiftDragPlugin

File: src/drone_description/urdf/construction_drone.xacro (robot description, xacro)
@@ -6,18 +6,16 @@
   <xacro:include filename="$(find drone_description)/urdf/fisheye_camera.xacro"/>
   <xacro:include filename="$(find drone_description)/urdf/propeller.xacro" />
-  <!-- Instantiate base (already includes world_link and base_link) -->
-  <!-- No additional instantiation needed for drone_base.xacro -->
   <!-- Instantiate LiDARs -->
-  <xacro:robosense_airy_lidar name="lidar_right" parent="base_link" xyz="0.122 0.0 0.18" rpy="0 0 0"/>
-  <xacro:robosense_airy_lidar name="lidar_left" parent="base_link" xyz="-0.122 0.0 0.18" rpy="0 0 3.14159"/>
-  <!-- Instatiate Fisheye Cameras -->
-  <xacro:fisheye_camera name="fisheye_camera_front" parent="base_link" xyz="0.0 0.139 0.14" rpy="0 0 3.14159" hfov="2.094"/> <!-- 3.14159 -->
-  <xacro:fisheye_camera name="fisheye_camera_rear" parent="base_link" xyz="0.0 -0.139 0.14" rpy="0 0 0" hfov="2.094" />
-  <xacro:fisheye_camera name="fisheye_camera_below" parent="base_link" xyz="0.0 0.0 0.095" rpy="1.5708 0 0" hfov="2.094" />
+  <xacro:robosense_airy_lidar name="lidar_right" parent="chassis_link" xyz="0.122 0.0 0.18" rpy="0 0 0"/>
+  <xacro:robosense_airy_lidar name="lidar_left"  parent="chassis_link" xyz="-0.122 0.0 0.18" rpy="0 0 3.14159"/>
+  <!-- Instantiate Fisheye Cameras -->
+  <xacro:fisheye_camera name="fisheye_camera_front" parent="chassis_link" xyz="0.0 0.139 0.14" rpy="0 0 3.14159" hfov="2.094"/>
+  <xacro:fisheye_camera name="fisheye_camera_rear"  parent="chassis_link" xyz="0.0 -0.139 0.14" rpy="0 0 0" hfov="2.094"/>
+  <xacro:fisheye_camera name="fisheye_camera_below" parent="chassis_link" xyz="0.0 0.0 0.095" rpy="1.5708 0 0" hfov="2.094"/>
   <!-- Instantiate Propellers -->
-  <xacro:propeller name="front_right_prop" parent="base_link" xyz="0.1050 0.105 0.24122" rpy="0 0 0"/>
-  <xacro:propeller name="front_left_prop" parent="base_link" xyz="-0.105 0.105 0.24122" rpy="0 0 0"/>
-  <xacro:propeller name="rear_left_prop" parent="base_link" xyz="-0.105 -0.105 0.24122" rpy="0 0 0"/>
-  <xacro:propeller name="rear_right_prop" parent="base_link" xyz="0.105 -0.105 0.24122" rpy="0 0 0"/>
+  <xacro:propeller name="front_right_prop" parent="chassis_link" xyz="0.1050 0.105 0.24122" rpy="0 0 0"/>
+  <xacro:propeller name="front_left_prop"  parent="chassis_link" xyz="-0.105 0.105 0.24122" rpy="0 0 0"/>
+  <xacro:propeller name="rear_left_prop"   parent="chassis_link" xyz="-0.105 -0.105 0.24122" rpy="0 0 0"/>
+  <xacro:propeller name="rear_right_prop"  parent="chassis_link" xyz="0.105 -0.105 0.24122" rpy="0 0 0"/>
   <!-- Gazebo plugin to enable ROS control -->
   <gazebo>
@@ -26,5 +24,5 @@
     </plugin>
   </gazebo>
-  <!-- Front Right Propeller Transmission -->
+  <!-- Propeller transmissions -->
   <transmission name="front_right_prop_transmission">
     <type>transmission_interface/SimpleTransmission</type>
@@ -37,5 +35,4 @@
     </actuator>
   </transmission>
-  <!-- Front Left Propeller Transmission -->
   <transmission name="front_left_prop_transmission">
     <type>transmission_interface/SimpleTransmission</type>
@@ -48,5 +45,4 @@
     </actuator>
   </transmission>
-  <!-- Rear Left Propeller Transmission -->
   <transmission name="rear_left_prop_transmission">
     <type>transmission_interface/SimpleTransmission</type>
@@ -59,5 +55,4 @@
     </actuator>
   </transmission>
-  <!-- Rear Right Propeller Transmission -->
   <transmission name="rear_right_prop_transmission">
     <type>transmission_interface/SimpleTransmission</type>
@@ -70,3 +65,45 @@
     </actuator>
   </transmission>
+  <!-- LiftDragPlugin: generates lift from joint velocity -->
+  <gazebo>
+    <plugin name="liftdrag_front_right" filename="libLiftDragPlugin.so">
+      <link_name>front_right_prop_link</link_name>
+      <control_joint>front_right_prop_joint</control_joint>
+      <a0>0.1</a0>
+      <cla>2.0</cla>
+      <cda>0.01</cda>
+      <area>1.2</area>
+      <air_density>1.225</air_density>
+      <cp>0 0 0</cp>
+      <forward>1 0 0</forward>
+      <upward>0 0 1</upward>
+    </plugin>
+  </gazebo>
+  <gazebo>
+    <plugin name="liftdrag_front_left" filename="libLiftDragPlugin.so">
+      <link_name>front_left_prop_link</link_name>
+      <control_joint>front_left_prop_joint</control_joint>
+      <a0>0.1</a0><cla>2.0</cla><cda>0.01</cda><area>1.2</area><air_density>1.225</air_density>
+      <cp>0 0 0</cp>
+      <forward>1 0 0</forward><upward>0 0 1</upward>
+    </plugin>
+  </gazebo>
+  <gazebo>
+    <plugin name="liftdrag_rear_left" filename="libLiftDragPlugin.so">
+      <link_name>rear_left_prop_link</link_name>
+      <control_joint>rear_left_prop_joint</control_joint>
+      <a0>0.1</a0><cla>2.0</cla><cda>0.01</cda><area>1.2</area><air_density>1.225</air_density>
+      <cp>0 0 0</cp>
+      <forward>1 0 0</forward><upward>0 0 1</upward>
+    </plugin>
+  </gazebo>
+  <gazebo>
+    <plugin name="liftdrag_rear_right" filename="libLiftDragPlugin.so">
+      <link_name>rear_right_prop_link</link_name>
+      <control_joint>rear_right_prop_joint</control_joint>
+      <a0>0.1</a0><cla>2.0</cla><cda>0.01</cda><area>1.2</area><air_density>1.225</air_density>
+      <cp>0 0 0</cp>
+      <forward>1 0 0</forward><upward>0 0 1</upward>
+    </plugin>
+  </gazebo>
 </robot>

File: src/drone_description/urdf/drone_base.xacro (robot description, xacro)
@@ -2,7 +2,7 @@
 <robot name="drone_base" xmlns:xacro="http://www.ros.org/wiki/xacro">
   <!-- Dummy root link to satisfy KDL (no inertia) -->
-  <link name="world_link"/>
+  <link name="base_link"/>
   <!-- Base link (drone chassis) -->
-  <link name="base_link">
+  <link name="chassis_link">
     <visual>
       <origin xyz="0 0 0.1" rpy="0 0 0"/>
@@ -17,6 +17,6 @@
       <origin xyz="0 0 0.1" rpy="0 0 0"/>
       <geometry>
-        <mesh filename="package://drone_description/meshes/drone_base_w_motors.stl" scale="1 1 1"/>
-        <!-- <box size="0.3 0.3 0.25"/>  -->
+        <!-- <mesh filename="package://drone_description/meshes/drone_base_w_motors.stl" scale="1 1 1"/>  -->
+        <box size="0.3 0.3 0.3"/>
       </geometry>
     </collision>
@@ -27,7 +27,7 @@
   </link>
   <!-- Fixed joint connecting world_link to base_link -->
-  <joint name="world_to_base" type="fixed">
-    <parent link="world_link"/>
-    <child link="base_link"/>
+  <joint name="base_to_chassis" type="fixed">
+    <parent link="base_link"/>
+    <child link="chassis_link"/>
     <origin xyz="0 0 0" rpy="0 0 0"/>
   </joint>
