Commit message: feat: add and configure r3live mapping in simulation

File: src/drone_description/urdf/construction_drone_hector.xacro (robot description, xacro)
@@ -7,9 +7,17 @@
   <xacro:include filename="$(find drone_description)/urdf/propeller.xacro"/>
   <!-- instantiate sensors as before -->
-  <xacro:robosense_airy_lidar name="lidar_right" parent="base_link" xyz="0.122 0.0 0.18" rpy="0 0 0"/>
+  <!-- <xacro:robosense_airy_lidar name="lidar_right" parent="base_link" xyz="0.122 0.0 0.18" rpy="0 0 0"/>
   <xacro:robosense_airy_lidar name="lidar_left"  parent="base_link" xyz="-0.122 0.0 0.18" rpy="0 0 3.14159"/>
-  <xacro:fisheye_camera name="fisheye_camera_front" parent="base_link" xyz="0.0 0.139 0.14" rpy="0 0 3.14159" hfov="2.094"/>
-  <xacro:fisheye_camera name="fisheye_camera_rear"  parent="base_link" xyz="0.0 -0.139 0.14" rpy="0 0 0" hfov="2.094"/>
-  <xacro:fisheye_camera name="fisheye_camera_below" parent="base_link" xyz="0.0 0.0 0.095" rpy="1.5708 0 0" hfov="2.094"/>
+  <xacro:fisheye_camera name="fisheye_camera_front" parent="base_link" xyz="0.0 0.139 0.14" rpy="0 0 3.14159" hfov="3.1415"/>
+  <xacro:fisheye_camera name="fisheye_camera_rear"  parent="base_link" xyz="0.0 -0.139 0.14" rpy="0 0 0" hfov="3.1415"/> -->
+  <!-- <xacro:fisheye_camera name="fisheye_camera_below" parent="base_link" xyz="0.0 0.0 0.095" rpy="1.5708 0 0" hfov="3.1415"/> -->
+  <!-- <xacro:robosense_airy_lidar name="lidar_right" parent="base_link" xyz="0.0 -0.139 0.14" rpy="0 0 0" />
+  <xacro:robosense_airy_lidar name="lidar_left" parent="base_link" xyz="0.0 0.139 0.14" rpy="0 0 3.14159" />
+  <xacro:fisheye_camera name="fisheye_camera_front" parent="base_link" xyz="-0.122 0.0 0.18" rpy="0 0 3.14159" hfov="3.1415"/>
+  <xacro:fisheye_camera name="fisheye_camera_rear" parent="base_link" xyz="0.122 0.0 0.18" rpy="0 0 0" hfov="3.1415"/> -->
+  <xacro:robosense_airy_lidar name="lidar_right" parent="base_link" xyz="0.0 -0.139 0.14" rpy="0 0 -1.5708"/>
+<xacro:robosense_airy_lidar name="lidar_left"  parent="base_link" xyz="0.0 0.139 0.14" rpy="0 0 1.5708"/>
+<!-- <xacro:fisheye_camera name="fisheye_camera_rear" parent="base_link" xyz="-0.122 0.0 0.18" rpy="0 0 -1.5708" hfov="3.1415"/> -->
+<xacro:fisheye_camera name="fisheye_camera_front"  parent="base_link" xyz="0.122 0.0 0.18" rpy="0 0 1.5708" hfov="3.1415"/>
   <!-- props, visual only (NO ros_control joints here) -->
   <xacro:propeller name="front_right_prop" parent="base_link" xyz="0.105  0.105  0.24122" rpy="0 0 0"/>
@@ -21,12 +29,12 @@
   <xacro:arg name="base_link_frame" default="base_link"/>
   <!-- include the exact Hector macro files we inspected -->
-  <!-- <xacro:include filename="$(find hector_quadrotor_gazebo)/urdf/quadrotor_controller.gazebo.xacro"/>
+  <xacro:include filename="$(find hector_quadrotor_gazebo)/urdf/quadrotor_controller.gazebo.xacro"/>
   <xacro:include filename="$(find hector_quadrotor_gazebo)/urdf/quadrotor_propulsion.gazebo.xacro"/>
   <xacro:include filename="$(find hector_quadrotor_gazebo)/urdf/quadrotor_aerodynamics.gazebo.xacro"/>
-  <xacro:include filename="$(find hector_quadrotor_gazebo)/urdf/quadrotor_sensors.gazebo.xacro" /> -->
+  <xacro:include filename="$(find hector_quadrotor_gazebo)/urdf/quadrotor_sensors.gazebo.xacro" />2
   <!-- call the macros (these inject the plugins) -->
-  <!-- <xacro:quadrotor_controller/>
+  <xacro:quadrotor_controller/>
   <xacro:quadrotor_propulsion/>
   <xacro:quadrotor_aerodynamics/>
-  <xacro:quadrotor_sensors/> -->
+  <xacro:quadrotor_sensors/>
 </robot>

File: src/drone_description/urdf/drone_base.xacro (robot description, xacro)
@@ -6,5 +6,5 @@
   <link name="base_link">
     <visual>
-      <origin xyz="0 0 0.1" rpy="0 0 0"/>
+      <origin xyz="0 0 0.1" rpy="0 0 0"/> <!-- 1.5708 -->
       <geometry>
         <mesh filename="package://drone_description/meshes/drone_base_w_motors.stl" scale="1 1 1"/> <!-- DAE mesh, assuming mm units -->

File: src/drone_description/urdf/fisheye_camera.xacro (robot description, xacro)
@@ -29,15 +29,15 @@
       <origin xyz="${xyz}" rpy="${rpy}"/>
     </joint>
-    <!-- Gazebo plugin for regular camera (not fisheye) -->
+    <!-- Wide-angle (fisheye) Gazebo sensor -->
     <gazebo reference="${name}_link">
-      <sensor type="camera" name="${name}_regular_cam">
+      <sensor type="wideanglecamera" name="${name}_fisheye_cam">
         <pose>0 -0.5 0 0 0 -1.5708</pose>
         <always_on>true</always_on>
-        <update_rate>30</update_rate>
+        <update_rate>50</update_rate>
         <camera>
           <horizontal_fov>${hfov}</horizontal_fov>
           <image>
-            <width>640</width>
-            <height>480</height>
+            <width>1280</width>
+            <height>720</height>
             <format>R8G8B8</format>
           </image>
@@ -46,11 +46,33 @@
             <far>100</far>
           </clip>
+          <distortion>
+            <k1>-0.28</k1>
+            <k2>0.074</k2>
+            <k3>0.0</k3>
+            <p1>0.0</p1>
+            <p2>0.0</p2>
+            <center>
+              <x>0.5</x>
+              <y>0.5</y>
+            </center>
+          </distortion>
+          <noise>
+            <type>gaussian</type>
+            <mean>0.0</mean>
+            <stddev>0.005</stddev>
+          </noise>
+          <lens>
+            <type>stereographic</type> or gnomonic, equidistant, etc.
+            <scale_to_hfov>true</scale_to_hfov>
+            <cutoff_angle>1.5708</cutoff_angle> 90 degrees
+            <env_texture_size>512</env_texture_size>
+          </lens>
         </camera>
         <plugin name="${name}_camera_controller" filename="libgazebo_ros_camera.so">
           <cameraName>${name}</cameraName>
-          <imageTopicName>${name}/image_raw</imageTopicName>
-          <cameraInfoTopicName>${name}/camera_info</cameraInfoTopicName>
+          <imageTopicName>/camera/image_color</imageTopicName>
+          <cameraInfoTopicName>/camera/camera_info</cameraInfoTopicName>
           <frameName>${name}_link</frameName>
-          <updateRate>30.0</updateRate>
+          <updateRate>50.0</updateRate>
         </plugin>
       </sensor>

Commit message: feat: add routine package to simplify launching and make it configurable

File: src/drone_description/urdf/construction_drone_hector.xacro (robot description, xacro)
@@ -1,9 +1,11 @@
 <?xml version="1.0"?>
 <robot name="construction_drone" xmlns:xacro="http://www.ros.org/wiki/xacro">
-  <!-- your model pieces -->
+  <xacro:arg name="simulation_mode" default="true"/>
   <xacro:include filename="$(find drone_description)/urdf/drone_base.xacro"/>
   <xacro:include filename="$(find drone_description)/urdf/airy_lidar.xacro"/>
   <xacro:include filename="$(find drone_description)/urdf/fisheye_camera.xacro"/>
   <xacro:include filename="$(find drone_description)/urdf/propeller.xacro"/>
+  <xacro:include filename="$(find drone_description)/urdf/plugins/airy_lidar_gazebo.xacro"/>
+  <xacro:include filename="$(find drone_description)/urdf/plugins/fisheye_camera_gazebo.xacro" />
   <!-- instantiate sensors as before -->
   <!-- <xacro:robosense_airy_lidar name="lidar_right" parent="base_link" xyz="0.122 0.0 0.18" rpy="0 0 0"/>
@@ -17,7 +19,24 @@
   <xacro:fisheye_camera name="fisheye_camera_rear" parent="base_link" xyz="0.122 0.0 0.18" rpy="0 0 0" hfov="3.1415"/> -->
   <xacro:robosense_airy_lidar name="lidar_right" parent="base_link" xyz="0.0 -0.139 0.14" rpy="0 0 -1.5708"/>
-<xacro:robosense_airy_lidar name="lidar_left"  parent="base_link" xyz="0.0 0.139 0.14" rpy="0 0 1.5708"/>
-<!-- <xacro:fisheye_camera name="fisheye_camera_rear" parent="base_link" xyz="-0.122 0.0 0.18" rpy="0 0 -1.5708" hfov="3.1415"/> -->
-<xacro:fisheye_camera name="fisheye_camera_front"  parent="base_link" xyz="0.122 0.0 0.18" rpy="0 0 1.5708" hfov="3.1415"/>
+  <xacro:robosense_airy_lidar name="lidar_left"  parent="base_link" xyz="0.0 0.139 0.14" rpy="0 0 1.5708"/>
+  <!-- <xacro:fisheye_camera name="fisheye_camera_rear" parent="base_link" xyz="-0.122 0.0 0.18" rpy="0 0 -1.5708" hfov="3.1415"/> -->
+  <xacro:fisheye_camera name="fisheye_camera_front"  parent="base_link" xyz="0.122 0.0 0.18" rpy="0 0 1.5708" />
+  <xacro:if value="$(arg simulation_mode)">
+    <xacro:robosense_airy_lidar_gazebo name="lidar_right" topic="/lidar_right/points" frame="lidar_right_link" />
+    <xacro:robosense_airy_lidar_gazebo name="lidar_left" topic="/lidar_left/points" frame="lidar_left_link" />
+    <xacro:fisheye_camera_gazebo name="fisheye_camera_front" topic="/camera/image_color" info_topic="/camera/camera_info" hfov="3.1415"/>
+    <xacro:arg name="world_frame" default="world"/>
+    <xacro:arg name="base_link_frame" default="base_link"/>
+    <!-- include the exact Hector macro files we inspected -->
+    <xacro:include filename="$(find hector_quadrotor_gazebo)/urdf/quadrotor_controller.gazebo.xacro"/>
+    <xacro:include filename="$(find hector_quadrotor_gazebo)/urdf/quadrotor_propulsion.gazebo.xacro"/>
+    <xacro:include filename="$(find hector_quadrotor_gazebo)/urdf/quadrotor_aerodynamics.gazebo.xacro"/>
+    <xacro:include filename="$(find hector_quadrotor_gazebo)/urdf/quadrotor_sensors.gazebo.xacro" />2
+    <!-- call the macros (these inject the plugins) -->
+    <xacro:quadrotor_controller/>
+    <xacro:quadrotor_propulsion/>
+    <xacro:quadrotor_aerodynamics/>
+    <xacro:quadrotor_sensors/>
+  </xacro:if>
   <!-- props, visual only (NO ros_control joints here) -->
   <xacro:propeller name="front_right_prop" parent="base_link" xyz="0.105  0.105  0.24122" rpy="0 0 0"/>
@@ -25,16 +44,3 @@
   <xacro:propeller name="rear_left_prop"   parent="base_link" xyz="-0.105 -0.105  0.24122" rpy="0 0 0"/>
   <xacro:propeller name="rear_right_prop"  parent="base_link" xyz="0.105  -0.105  0.24122" rpy="0 0 0"/>
-  <!-- make the same args Hector's macros expect -->
-  <xacro:arg name="world_frame" default="world"/>
-  <xacro:arg name="base_link_frame" default="base_link"/>
-  <!-- include the exact Hector macro files we inspected -->
-  <xacro:include filename="$(find hector_quadrotor_gazebo)/urdf/quadrotor_controller.gazebo.xacro"/>
-  <xacro:include filename="$(find hector_quadrotor_gazebo)/urdf/quadrotor_propulsion.gazebo.xacro"/>
-  <xacro:include filename="$(find hector_quadrotor_gazebo)/urdf/quadrotor_aerodynamics.gazebo.xacro"/>
-  <xacro:include filename="$(find hector_quadrotor_gazebo)/urdf/quadrotor_sensors.gazebo.xacro" />2
-  <!-- call the macros (these inject the plugins) -->
-  <xacro:quadrotor_controller/>
-  <xacro:quadrotor_propulsion/>
-  <xacro:quadrotor_aerodynamics/>
-  <xacro:quadrotor_sensors/>
 </robot>

File: src/drone_description/urdf/fisheye_camera.xacro (robot description, xacro)
@@ -2,5 +2,5 @@
 <robot name="fisheye_camera" xmlns:xacro="http://www.ros.org/wiki/xacro">
   <!-- Macro for wide-angle (fisheye) camera -->
-  <xacro:macro name="fisheye_camera" params="name parent xyz rpy hfov">
+  <xacro:macro name="fisheye_camera" params="name parent xyz rpy">
     <link name="${name}_link">
       <visual>
@@ -30,5 +30,5 @@
     </joint>
     <!-- Wide-angle (fisheye) Gazebo sensor -->
-    <gazebo reference="${name}_link">
+    <!-- <gazebo reference="${name}_link">
       <sensor type="wideanglecamera" name="${name}_fisheye_cam">
         <pose>0 -0.5 0 0 0 -1.5708</pose>
@@ -77,5 +77,5 @@
         </plugin>
       </sensor>
-    </gazebo>
+    </gazebo> -->
   </xacro:macro>
 </robot>

Commit message: fix: rear and front camera extrinsics

File: src/drone_description/urdf/construction_drone_hector.xacro (robot description, xacro)
@@ -8,29 +8,32 @@
   <xacro:include filename="$(find drone_description)/urdf/plugins/airy_lidar_gazebo.xacro"/>
   <xacro:include filename="$(find drone_description)/urdf/plugins/fisheye_camera_gazebo.xacro" />
-  <!-- instantiate sensors as before -->
+  <!-- First positioning -->
   <!-- <xacro:robosense_airy_lidar name="lidar_right" parent="base_link" xyz="0.122 0.0 0.18" rpy="0 0 0"/>
   <xacro:robosense_airy_lidar name="lidar_left"  parent="base_link" xyz="-0.122 0.0 0.18" rpy="0 0 3.14159"/>
-  <xacro:fisheye_camera name="fisheye_camera_front" parent="base_link" xyz="0.0 0.139 0.14" rpy="0 0 3.14159" hfov="3.1415"/>
-  <xacro:fisheye_camera name="fisheye_camera_rear"  parent="base_link" xyz="0.0 -0.139 0.14" rpy="0 0 0" hfov="3.1415"/> -->
-  <!-- <xacro:fisheye_camera name="fisheye_camera_below" parent="base_link" xyz="0.0 0.0 0.095" rpy="1.5708 0 0" hfov="3.1415"/> -->
+  <xacro:fisheye_camera name="fisheye_camera_front" parent="base_link" xyz="0.0 0.139 0.14" rpy="0 0 3.14159" /> -->
+  <!-- <xacro:fisheye_camera name="fisheye_camera_rear"  parent="base_link" xyz="0.0 -0.139 0.14" rpy="0 0 0" hfov="3.1415"/> -->
+  <!-- <xacro:fisheye_camera name="fisheye_camera_below" parent="base_link" xyz="0.0 0.0 0.095" rpy="1.5708 0 0" /> -->
   <!-- <xacro:robosense_airy_lidar name="lidar_right" parent="base_link" xyz="0.0 -0.139 0.14" rpy="0 0 0" />
   <xacro:robosense_airy_lidar name="lidar_left" parent="base_link" xyz="0.0 0.139 0.14" rpy="0 0 3.14159" />
   <xacro:fisheye_camera name="fisheye_camera_front" parent="base_link" xyz="-0.122 0.0 0.18" rpy="0 0 3.14159" hfov="3.1415"/>
   <xacro:fisheye_camera name="fisheye_camera_rear" parent="base_link" xyz="0.122 0.0 0.18" rpy="0 0 0" hfov="3.1415"/> -->
+  <!-- Second positioning -->
   <xacro:robosense_airy_lidar name="lidar_right" parent="base_link" xyz="0.0 -0.139 0.14" rpy="0 0 -1.5708"/>
   <xacro:robosense_airy_lidar name="lidar_left"  parent="base_link" xyz="0.0 0.139 0.14" rpy="0 0 1.5708"/>
-  <!-- <xacro:fisheye_camera name="fisheye_camera_rear" parent="base_link" xyz="-0.122 0.0 0.18" rpy="0 0 -1.5708" hfov="3.1415"/> -->
   <xacro:fisheye_camera name="fisheye_camera_front"  parent="base_link" xyz="0.122 0.0 0.18" rpy="0 0 1.5708" />
+  <!-- <xacro:fisheye_camera name="fisheye_camera_rear" parent="base_link" xyz="-0.122 0.0 0.18" rpy="0 0 -1.5708" /> -->
   <xacro:if value="$(arg simulation_mode)">
-    <xacro:robosense_airy_lidar_gazebo name="lidar_right" topic="/lidar_right/points" frame="lidar_right_link" />
-    <xacro:robosense_airy_lidar_gazebo name="lidar_left" topic="/lidar_left/points" frame="lidar_left_link" />
+    <xacro:robosense_airy_lidar_gazebo name="lidar_right" topic="/lidar_right/points" pose="0.0 0.0 0.0 0.0 0.0 0.0"/>
+    <xacro:robosense_airy_lidar_gazebo name="lidar_left" topic="/lidar_left/points" pose="0.0 0.0 0.0 0.0 0.0 0.0"/>
     <xacro:fisheye_camera_gazebo name="fisheye_camera_front" topic="/camera/image_color" info_topic="/camera/camera_info" hfov="3.1415"/>
+    <!-- <xacro:fisheye_camera_gazebo name="fisheye_camera_rear" topic="/camera/image_color" info_topic="/camera/camera_info" hfov="3.1415"/> -->
+    <!-- <xacro:fisheye_camera_gazebo name="fisheye_camera_below" topic="/camera/image_color" info_topic="/camera/camera_info" hfov="3.1415"/> -->
     <xacro:arg name="world_frame" default="world"/>
-    <xacro:arg name="base_link_frame" default="base_link"/>
+    <xacro:arg name="base_link_frame" default="lidar_left_link"/>
     <!-- include the exact Hector macro files we inspected -->
     <xacro:include filename="$(find hector_quadrotor_gazebo)/urdf/quadrotor_controller.gazebo.xacro"/>
     <xacro:include filename="$(find hector_quadrotor_gazebo)/urdf/quadrotor_propulsion.gazebo.xacro"/>
     <xacro:include filename="$(find hector_quadrotor_gazebo)/urdf/quadrotor_aerodynamics.gazebo.xacro"/>
-    <xacro:include filename="$(find hector_quadrotor_gazebo)/urdf/quadrotor_sensors.gazebo.xacro" />2
+    <xacro:include filename="$(find hector_quadrotor_gazebo)/urdf/quadrotor_sensors.gazebo.xacro" />
     <!-- call the macros (these inject the plugins) -->
     <xacro:quadrotor_controller/>

File: src/drone_description/urdf/drone_base.xacro (robot description, xacro)
@@ -8,5 +8,5 @@
       <origin xyz="0 0 0.1" rpy="0 0 0"/> <!-- 1.5708 -->
       <geometry>
-        <mesh filename="package://drone_description/meshes/drone_base_w_motors.stl" scale="1 1 1"/> <!-- DAE mesh, assuming mm units -->
+        <mesh filename="package://drone_description/meshes/drone_base_complete.stl" scale="1 1 1"/> <!-- DAE mesh, assuming mm units -->
       </geometry>
       <material name="blue">

File: src/drone_description/urdf/fisheye_camera.xacro (robot description, xacro)
@@ -28,4 +28,11 @@
       <child link="${name}_link"/>
       <origin xyz="${xyz}" rpy="${rpy}"/>
+    </joint>
+    <link name="${name}_optical_frame"/>
+    <joint name="${name}_optical_from_link" type="fixed">
+      <parent link="${name}_link"/>
+      <child  link="${name}_optical_frame"/>
+      <!-- camera_link -> camera_optical (OpenCV) -->
+      <origin xyz="0 0 0" rpy="-1.57079632679 0 -1.57079632679"/>
     </joint>
     <!-- Wide-angle (fisheye) Gazebo sensor -->

File: src/drone_description/urdf/plugins/airy_lidar_gazebo.xacro (robot description, xacro)
@@ -2,8 +2,8 @@
 <robot name="robosense_airy_lidar_gz" xmlns:xacro="http://www.ros.org/wiki/xacro">
   <!-- Gazebo sensor + ROS plugin for the Robosense Airy LIDAR -->
-  <xacro:macro name="robosense_airy_lidar_gazebo" params="name frame topic">
-    <gazebo reference="${frame}">
+  <xacro:macro name="robosense_airy_lidar_gazebo" params="name topic pose">
+    <gazebo reference="${name}_link">
       <sensor type="gpu_ray" name="${name}_velodyne">
-        <pose>0 0 0 0 0 0</pose>
+        <pose>${pose}</pose>
         <update_rate>20</update_rate>
         <visualize>true</visualize>
@@ -31,5 +31,5 @@
         <plugin name="${name}_plugin" filename="libgazebo_ros_velodyne_gpu_laser.so">
           <topicName>${topic}</topicName>
-          <frameName>${frame}</frameName>
+          <frameName>${name}_link</frameName>
         </plugin>
       </sensor>

File: src/external_pkgs/hector-quadrotor-noetic/hector_quadrotor/hector_quadrotor_gazebo/urdf/quadrotor_sensors.gazebo.xacro (robot description, xacro)
@@ -6,5 +6,7 @@
           <plugin name="quadrotor_imu_sim" filename="libhector_gazebo_ros_imu.so">
             <updateRate>100.0</updateRate>
-            <bodyName>base_link</bodyName>
+            <!-- <bodyName>base_link</bodyName> -->
+            <!-- <frameId>$(arg base_link_frame)</frameId> -->
+            <bodyName>$(arg base_link_frame)</bodyName>
             <frameId>$(arg base_link_frame)</frameId>
             <topicName>raw_imu</topicName>
@@ -18,5 +20,6 @@
           <plugin name="quadrotor_baro_sim" filename="libhector_gazebo_ros_baro.so">
             <updateRate>10.0</updateRate>
-            <bodyName>base_link</bodyName>
+            <!-- <bodyName>base_link</bodyName> -->
+            <bodyName>$(arg base_link_frame)</bodyName>
             <frameId>$(arg base_link_frame)</frameId>
             <topicName>pressure_height</topicName>
@@ -28,5 +31,6 @@
           <plugin name="quadrotor_magnetic_sim" filename="libhector_gazebo_ros_magnetic.so">
             <updateRate>10.0</updateRate>
-            <bodyName>base_link</bodyName>
+            <!-- <bodyName>base_link</bodyName> -->
+            <bodyName>$(arg base_link_frame)</bodyName>
             <frameId>$(arg base_link_frame)</frameId>
             <topicName>magnetic</topicName>
@@ -37,5 +41,6 @@
           <plugin name="quadrotor_gps_sim" filename="libhector_gazebo_ros_gps.so">
             <updateRate>4.0</updateRate>
-            <bodyName>base_link</bodyName>
+            <!-- <bodyName>base_link</bodyName> -->
+            <bodyName>$(arg base_link_frame)</bodyName>
             <frameId>$(arg base_link_frame)</frameId>
             <topicName>fix</topicName>
@@ -50,5 +55,6 @@
           <plugin name="quadrotor_groundtruth_sim" filename="libgazebo_ros_p3d.so">
             <updateRate>100.0</updateRate>
-            <bodyName>base_link</bodyName>
+            <!-- <bodyName>base_link</bodyName> -->
+            <bodyName>$(arg base_link_frame)</bodyName>
             <topicName>ground_truth/state</topicName>
             <gaussianNoise>0.0</gaussianNoise>
