Commit message: feat(WIP): add propeller plugins in gazebo

File: src/drone_description/urdf/airy_lidar.xacro (robot description, xacro)
@@ -30,5 +30,5 @@
     </joint>
     <!-- Gazebo Sensor -->
-    <gazebo reference="${name}_link">
+    <!-- <gazebo reference="${name}_link">
       <sensor type="gpu_ray" name="${name}_velodyne">
         <pose>0 0 0 0 0 0</pose>
@@ -61,5 +61,5 @@
         </plugin>
       </sensor>
-    </gazebo>
+    </gazebo> -->
     </xacro:macro>
     <!-- Gazebo Reference -->

File: src/drone_description/urdf/construction_drone.xacro (robot description, xacro)
@@ -4,7 +4,6 @@
   <xacro:include filename="$(find drone_description)/urdf/drone_base.xacro"/>
   <xacro:include filename="$(find drone_description)/urdf/airy_lidar.xacro"/>
-  <!-- <xacro:include filename="$(find drone_description)/urdf/airy_lidar_left.xacro"/> -->
   <xacro:include filename="$(find drone_description)/urdf/fisheye_camera.xacro"/>
-  <!-- <xacro:include filename="$(find drone_description)/urdf/fisheye_camera_rear.xacro"/> -->
+  <xacro:include filename="$(find drone_description)/urdf/propeller.xacro" />
   <!-- Instantiate base (already includes world_link and base_link) -->
   <!-- No additional instantiation needed for drone_base.xacro -->
@@ -16,3 +15,52 @@
   <xacro:fisheye_camera name="fisheye_camera_rear" parent="base_link" xyz="0.0 -0.139 0.14" rpy="0 0 0" hfov="2.094" />
   <xacro:fisheye_camera name="fisheye_camera_below" parent="base_link" xyz="0.0 0.0 0.095" rpy="1.5708 0 0" hfov="2.094" />
+  <!-- Instantiate Propellers -->
+  <xacro:propeller name="front_right_prop" parent="base_link" xyz="0.1050 0.105 0.24122" rpy="0 0 0"/>
+  <xacro:propeller name="front_left_prop" parent="base_link" xyz="-0.105 0.105 0.24122" rpy="0 0 0"/>
+  <xacro:propeller name="rear_left_prop" parent="base_link" xyz="-0.105 -0.105 0.24122" rpy="0 0 0"/>
+  <xacro:propeller name="rear_right_prop" parent="base_link" xyz="0.105 -0.105 0.24122" rpy="0 0 0"/>
+  <!-- Front Right Propeller Transmission -->
+  <transmission name="front_right_prop_transmission">
+    <type>transmission_interface/SimpleTransmission</type>
+    <joint name="front_right_prop_joint">
+      <hardwareInterface>EffortJointInterface</hardwareInterface>
+    </joint>
+    <actuator name="front_right_prop_motor">
+      <hardwareInterface>EffortJointInterface</hardwareInterface>
+      <mechanicalReduction>1</mechanicalReduction>
+    </actuator>
+  </transmission>
+  <!-- Front Left Propeller Transmission -->
+  <transmission name="front_left_prop_transmission">
+    <type>transmission_interface/SimpleTransmission</type>
+    <joint name="front_left_prop_joint">
+      <hardwareInterface>EffortJointInterface</hardwareInterface>
+    </joint>
+    <actuator name="front_left_prop_motor">
+      <hardwareInterface>EffortJointInterface</hardwareInterface>
+      <mechanicalReduction>1</mechanicalReduction>
+    </actuator>
+  </transmission>
+  <!-- Rear Left Propeller Transmission -->
+  <transmission name="rear_left_prop_transmission">
+    <type>transmission_interface/SimpleTransmission</type>
+    <joint name="rear_left_prop_joint">
+      <hardwareInterface>EffortJointInterface</hardwareInterface>
+    </joint>
+    <actuator name="rear_left_prop_motor">
+      <hardwareInterface>EffortJointInterface</hardwareInterface>
+      <mechanicalReduction>1</mechanicalReduction>
+    </actuator>
+  </transmission>
+  <!-- Rear Right Propeller Transmission -->
+  <transmission name="rear_right_prop_transmission">
+    <type>transmission_interface/SimpleTransmission</type>
+    <joint name="rear_right_prop_joint">
+      <hardwareInterface>EffortJointInterface</hardwareInterface>
+    </joint>
+    <actuator name="rear_right_prop_motor">
+      <hardwareInterface>EffortJointInterface</hardwareInterface>
+      <mechanicalReduction>1</mechanicalReduction>
+    </actuator>
+  </transmission>
 </robot>

File: src/drone_description/urdf/drone_base.xacro (robot description, xacro)
@@ -8,5 +8,5 @@
       <origin xyz="0 0 0.1" rpy="0 0 0"/>
       <geometry>
-        <mesh filename="package://drone_description/meshes/drone_base.dae" scale="1 1 1"/> <!-- DAE mesh, assuming mm units -->
+        <mesh filename="package://drone_description/meshes/drone_base_with_motors.dae" scale="1 1 1"/> <!-- DAE mesh, assuming mm units -->
       </geometry>
       <material name="blue">
@@ -15,8 +15,8 @@
     </visual>
     <collision>
-      <origin xyz="0 0 0" rpy="0 0 0"/>
+      <origin xyz="0 0 0.1" rpy="0 0 0"/>
       <geometry>
-        <!-- <mesh filename="package://drone_description/meshes/drone_base.dae" scale="0.001 0.001 0.001"/> Same mesh for collision -->
-        <box size="0.3 0.3 0.25"/> <!-- Placeholder box for collision, adjust size as needed -->
+        <mesh filename="package://drone_description/meshes/drone_base_with_motors.dae" scale="1 1 1"/>
+        <!-- <box size="0.3 0.3 0.25"/>  -->
       </geometry>
     </collision>

File: src/drone_description/urdf/fisheye_camera.xacro (robot description, xacro)
@@ -30,5 +30,5 @@
     </joint>
     <!-- Gazebo plugin for regular camera (not fisheye) -->
-    <gazebo reference="${name}_link">
+    <!-- <gazebo reference="${name}_link">
       <sensor type="camera" name="${name}_regular_cam">
         <pose>0 -0.5 0 0 0 -1.5708</pose>
@@ -55,5 +55,5 @@
         </plugin>
       </sensor>
-    </gazebo>
+    </gazebo> -->
   </xacro:macro>
 </robot>

Commit message: feat: fix gazebo flight simulation

File: src/drone_description/urdf/airy_lidar.xacro (robot description, xacro)
@@ -30,5 +30,5 @@
     </joint>
     <!-- Gazebo Sensor -->
-    <!-- <gazebo reference="${name}_link">
+    <gazebo reference="${name}_link">
       <sensor type="gpu_ray" name="${name}_velodyne">
         <pose>0 0 0 0 0 0</pose>
@@ -61,5 +61,5 @@
         </plugin>
       </sensor>
-    </gazebo> -->
+    </gazebo>
     </xacro:macro>
     <!-- Gazebo Reference -->

File: src/drone_description/urdf/construction_drone.xacro (robot description, xacro)
@@ -7,15 +7,15 @@
   <xacro:include filename="$(find drone_description)/urdf/propeller.xacro" />
   <!-- Instantiate LiDARs -->
-  <xacro:robosense_airy_lidar name="lidar_right" parent="chassis_link" xyz="0.122 0.0 0.18" rpy="0 0 0"/>
-  <xacro:robosense_airy_lidar name="lidar_left"  parent="chassis_link" xyz="-0.122 0.0 0.18" rpy="0 0 3.14159"/>
+  <xacro:robosense_airy_lidar name="lidar_right" parent="base_link" xyz="0.122 0.0 0.18" rpy="0 0 0"/>
+  <xacro:robosense_airy_lidar name="lidar_left"  parent="base_link" xyz="-0.122 0.0 0.18" rpy="0 0 3.14159"/>
   <!-- Instantiate Fisheye Cameras -->
-  <xacro:fisheye_camera name="fisheye_camera_front" parent="chassis_link" xyz="0.0 0.139 0.14" rpy="0 0 3.14159" hfov="2.094"/>
-  <xacro:fisheye_camera name="fisheye_camera_rear"  parent="chassis_link" xyz="0.0 -0.139 0.14" rpy="0 0 0" hfov="2.094"/>
-  <xacro:fisheye_camera name="fisheye_camera_below" parent="chassis_link" xyz="0.0 0.0 0.095" rpy="1.5708 0 0" hfov="2.094"/>
+  <xacro:fisheye_camera name="fisheye_camera_front" parent="base_link" xyz="0.0 0.139 0.14" rpy="0 0 3.14159" hfov="2.094"/>
+  <xacro:fisheye_camera name="fisheye_camera_rear"  parent="base_link" xyz="0.0 -0.139 0.14" rpy="0 0 0" hfov="2.094"/>
+  <xacro:fisheye_camera name="fisheye_camera_below" parent="base_link" xyz="0.0 0.0 0.095" rpy="1.5708 0 0" hfov="2.094"/>
   <!-- Instantiate Propellers -->
-  <xacro:propeller name="front_right_prop" parent="chassis_link" xyz="0.1050 0.105 0.24122" rpy="0 0 0"/>
-  <xacro:propeller name="front_left_prop"  parent="chassis_link" xyz="-0.105 0.105 0.24122" rpy="0 0 0"/>
-  <xacro:propeller name="rear_left_prop"   parent="chassis_link" xyz="-0.105 -0.105 0.24122" rpy="0 0 0"/>
-  <xacro:propeller name="rear_right_prop"  parent="chassis_link" xyz="0.105 -0.105 0.24122" rpy="0 0 0"/>
+  <xacro:propeller name="front_right_prop" parent="base_link" xyz="0.1050 0.105 0.24122" rpy="0 0 0"/>
+  <xacro:propeller name="front_left_prop"  parent="base_link" xyz="-0.105 0.105 0.24122" rpy="0 0 0"/>
+  <xacro:propeller name="rear_left_prop"   parent="base_link" xyz="-0.105 -0.105 0.24122" rpy="0 0 0"/>
+  <xacro:propeller name="rear_right_prop"  parent="base_link" xyz="0.105 -0.105 0.24122" rpy="0 0 0"/>
   <!-- Gazebo plugin to enable ROS control -->
   <gazebo>
@@ -71,11 +71,11 @@
       <control_joint>front_right_prop_joint</control_joint>
       <a0>0.1</a0>
-      <cla>2.0</cla>
+      <cla>4.0</cla>
       <cda>0.01</cda>
-      <area>1.2</area>
+      <area>2.0</area>
       <air_density>1.225</air_density>
       <cp>0 0 0</cp>
       <forward>1 0 0</forward>
-      <upward>0 0 1</upward>
+      <upward>0 0 -1</upward>
     </plugin>
   </gazebo>
@@ -84,5 +84,5 @@
       <link_name>front_left_prop_link</link_name>
       <control_joint>front_left_prop_joint</control_joint>
-      <a0>0.1</a0><cla>2.0</cla><cda>0.01</cda><area>1.2</area><air_density>1.225</air_density>
+      <a0>0.1</a0><cla>4.0</cla><cda>0.01</cda><area>2.0</area><air_density>1.225</air_density>
       <cp>0 0 0</cp>
       <forward>1 0 0</forward><upward>0 0 1</upward>
@@ -93,7 +93,7 @@
       <link_name>rear_left_prop_link</link_name>
       <control_joint>rear_left_prop_joint</control_joint>
-      <a0>0.1</a0><cla>2.0</cla><cda>0.01</cda><area>1.2</area><air_density>1.225</air_density>
+      <a0>0.1</a0><cla>4.0</cla><cda>0.01</cda><area>2.0</area><air_density>1.225</air_density>
       <cp>0 0 0</cp>
-      <forward>1 0 0</forward><upward>0 0 1</upward>
+      <forward>1 0 0</forward><upward>0 0 -1</upward>
     </plugin>
   </gazebo>
@@ -102,5 +102,5 @@
       <link_name>rear_right_prop_link</link_name>
       <control_joint>rear_right_prop_joint</control_joint>
-      <a0>0.1</a0><cla>2.0</cla><cda>0.01</cda><area>1.2</area><air_density>1.225</air_density>
+      <a0>0.1</a0><cla>4.0</cla><cda>0.01</cda><area>2.0</area><air_density>1.225</air_density>
       <cp>0 0 0</cp>
       <forward>1 0 0</forward><upward>0 0 1</upward>

File: src/drone_description/urdf/drone_base.xacro (robot description, xacro)
@@ -2,7 +2,7 @@
 <robot name="drone_base" xmlns:xacro="http://www.ros.org/wiki/xacro">
   <!-- Dummy root link to satisfy KDL (no inertia) -->
-  <link name="base_link"/>
+  <!-- <link name="base_link"/> -->
   <!-- Base link (drone chassis) -->
-  <link name="chassis_link">
+  <link name="base_link">
     <visual>
       <origin xyz="0 0 0.1" rpy="0 0 0"/>
@@ -18,5 +18,5 @@
       <geometry>
         <!-- <mesh filename="package://drone_description/meshes/drone_base_w_motors.stl" scale="1 1 1"/>  -->
-        <box size="0.3 0.3 0.3"/>
+        <box size="0.3 0.3 0.2"/>
       </geometry>
     </collision>
@@ -27,8 +27,8 @@
   </link>
   <!-- Fixed joint connecting world_link to base_link -->
-  <joint name="base_to_chassis" type="fixed">
+  <!-- <joint name="base_to_chassis" type="fixed">
     <parent link="base_link"/>
     <child link="chassis_link"/>
     <origin xyz="0 0 0" rpy="0 0 0"/>
-  </joint>
+  </joint> -->
 </robot>

File: src/drone_description/urdf/fisheye_camera.xacro (robot description, xacro)
@@ -30,5 +30,5 @@
     </joint>
     <!-- Gazebo plugin for regular camera (not fisheye) -->
-    <!-- <gazebo reference="${name}_link">
+    <gazebo reference="${name}_link">
       <sensor type="camera" name="${name}_regular_cam">
         <pose>0 -0.5 0 0 0 -1.5708</pose>
@@ -55,5 +55,5 @@
         </plugin>
       </sensor>
-    </gazebo> -->
+    </gazebo>
   </xacro:macro>
 </robot>

Commit message: feat: add drone 1 Lidar 1 camera configurations

File: src/drone_description/urdf/airy_lidar.xacro (robot description, xacro)
@@ -20,5 +20,5 @@
       </collision>
       <inertial>
-        <mass value="0.24"/>
+        <mass value="0.0"/>
         <inertia ixx="0.0001" ixy="0.0" ixz="0.0" iyy="0.0001" iyz="0.0" izz="0.0001"/>
       </inertial>

File: src/drone_description/urdf/drone_2L3C.xacro (robot description, xacro)
@@ -1,4 +1,4 @@
 <?xml version="1.0"?>
-<robot name="construction_drone" xmlns:xacro="http://www.ros.org/wiki/xacro">
+<robot name="drone_2L3C" xmlns:xacro="http://www.ros.org/wiki/xacro">
   <xacro:arg name="simulation_mode" default="true"/>
   <xacro:include filename="$(find drone_description)/urdf/drone_base.xacro"/>

File: src/drone_description/urdf/fisheye_camera.xacro (robot description, xacro)
@@ -20,5 +20,5 @@
       </collision>
       <inertial>
-        <mass value="0.05"/>
+        <mass value="0.0"/>
         <inertia ixx="0.00001" ixy="0.0" ixz="0.0" iyy="0.00001" iyz="0.0" izz="0.00001"/>
       </inertial>

File: src/drone_description/urdf/plugins/airy_lidar_gazebo.xacro (robot description, xacro)
@@ -7,5 +7,5 @@
         <pose>${pose}</pose>
         <update_rate>20</update_rate>
-        <visualize>true</visualize>
+        <visualize>true</visualize> <!-- set 'true' to make it visible in gazebo -->
         <ray>
           <scan>
